Commit message: Imported upstream version '2.1.0' of 'upstream'

File: talos_description/urdf/gripper/gripper.ros2_control.xacro (robot description, xacro)
@@ -14,25 +14,17 @@
 <robot xmlns:xacro="http://ros.org/wiki/xacro">
   <xacro:macro name="ros2_control_gripper" params="name" >
-    <!-- <xacro:macro name="ros2_control_talos_gripper_mimic_joint" params="mimic_joint_name actuated_joint_name multiplier" >
+    <xacro:macro name="ros2_control_talos_gripper_mimic_joint" params="mimic_joint_name actuated_joint_name multiplier" >
       <joint name="${mimic_joint_name}">
         <param name="mimic">${actuated_joint_name}</param>
         <param name="multiplier">${multiplier}</param>
-        <command_interface name="position" />
-        <command_interface name="velocity" />
-        <command_interface name="effort" />
-        <state_interface name="position"/>
-        <state_interface name="velocity" />
-        <state_interface name="effort" />
       </joint>
-    </xacro:macro> -->
+    </xacro:macro>
     <joint name="${name}_joint">
       <command_interface name="position" />
-      <command_interface name="velocity" />
-      <command_interface name="effort" />
-      <state_interface name="position" />
+      <state_interface name="position"/>
       <state_interface name="velocity" />
       <state_interface name="effort" />
     </joint>
-    <!-- <xacro:ros2_control_talos_gripper_mimic_joint mimic_joint_name="${name}_inner_double_joint"
+    <xacro:ros2_control_talos_gripper_mimic_joint mimic_joint_name="${name}_inner_double_joint"
                                                     actuated_joint_name="${name}_joint"
                                                     multiplier="1"/>
@@ -51,5 +43,5 @@
     <xacro:ros2_control_talos_gripper_mimic_joint mimic_joint_name="${name}_fingertip_3_joint"
                                                     actuated_joint_name="${name}_joint"
-                                                    multiplier="-1"/> -->
+                                                    multiplier="-1"/>
    <!-- transmissions -->
   <xacro:include filename="$(find talos_description)/urdf/gripper/gripper.transmission.xacro" />

File: talos_description/urdf/gripper/gripper.transmission.xacro (robot description, xacro)
@@ -18,16 +18,5 @@
       <actuator name="${name}_actuator" role="actuator1" />
       <joint name="${name}_joint" role="joint1">
-        <mechanicalReduction>${reduction}</mechanicalReduction>
-        <offset>0.0</offset>
-      </joint>
-    </transmission>
-  </xacro:macro>
-  <xacro:macro name="gripper_virtual_transmission" params="name reduction" >
-    <transmission name="${name}_trans">
-      <plugin>transmission_interface/SimpleTransmission</plugin>
-      <actuator name="${name}_actuator"  role="actuator1"/>
-      <joint name="${name}_joint" role="joint1">
-        <mechanicalReduction>${reduction}</mechanicalReduction>
-        <offset>0.0</offset>
+        <mechanical_reduction>${reduction}</mechanical_reduction>
       </joint>
     </transmission>

File: talos_description/urdf/head/head.transmission.xacro (robot description, xacro)
@@ -11,18 +11,18 @@
                params="name number1 number2 act_reduction1 act_reduction2 jnt_reduction1 jnt_reduction2 offset_value_1 offset_value_2" >
     <transmission name="talos_trans">
-      <plugin>transmission_interface/HalfDifferentialTransmission</plugin>
+      <plugin>pal_transmissions/HalfDifferentialTransmission</plugin>
       <actuator name="${name}_${number1}_actuator" role="actuator1">
-        <mechanicalReduction>${act_reduction1}</mechanicalReduction>
+        <mechanical_reduction>${act_reduction1}</mechanical_reduction>
       </actuator>
       <actuator name="${name}_${number2}_actuator" role="actuator2">
-        <mechanicalReduction>${act_reduction2}</mechanicalReduction>
+        <mechanical_reduction>${act_reduction2}</mechanical_reduction>
       </actuator>
       <joint name="${name}_${number1}_joint" role="joint1">
         <offset>${offset_value_1}</offset>
-        <mechanicalReduction>${jnt_reduction1}</mechanicalReduction>
+        <mechanical_reduction>${jnt_reduction1}</mechanical_reduction>
       </joint>
       <joint name="${name}_${number2}_joint" role="joint2">
         <offset>${offset_value_2}</offset>
-        <mechanicalReduction>${jnt_reduction2}</mechanicalReduction>
+        <mechanical_reduction>${jnt_reduction2}</mechanical_reduction>
       </joint>
     </transmission>
