Commit message: Imported upstream version '2.10.3' of 'upstream'

File: talos_description/ros2_control/ros2_control.urdf.xacro (robot description, xacro)
@@ -29,5 +29,5 @@
       <xacro:unless value="$(arg use_sim)">
         <properties>
-          <async thread_priority="70" affinity="[4]" scheduling_policy="detached"/>
+          <async thread_priority="70" affinity="[1]" scheduling_policy="detached"/>
         </properties>
       </xacro:unless>
@@ -39,4 +39,5 @@
           <plugin>robot_control/RobotControl</plugin>
           <param name="error_protection">true</param>
+          <param name="expose_safety_interface">true</param>
           <param name="idle_mode_on_stop">true</param>
           <param name="idle_mode_on_stop_interfaces">[current, effort, torque]</param>

File: talos_description/urdf/talos_full_common.urdf.xacro (robot description, xacro)
@@ -15,5 +15,7 @@
   <xacro:arg name="use_sim" default="false"/>
   <xacro:arg name="multiple" default="false"/>
+  <xacro:arg name="gazebo_version" default="classic"/>
   <xacro:property name="is_multiple" value="$(arg multiple)" />
+  <xacro:property name="gazebo_version" value="$(arg gazebo_version)" />
   <xacro:if value="$(arg enable_crane)">
     <xacro:include filename="$(find talos_description)/urdf/crane/crane.urdf.xacro" />
